Commit message: update xmlns + beautifying

File: frida_description/urdf/adapter.urdf.xacro (robot description, xacro)
@@ -1,15 +1,12 @@
 <?xml version="1.0"?>
-<robot xmlns:sensor="http://playerstage.sourceforge.net/gazebo/xmlschema/#sensor"
-       xmlns:controller="http://playerstage.sourceforge.net/gazebo/xmlschema/#controller"
-       xmlns:interface="http://playerstage.sourceforge.net/gazebo/xmlschema/#interface"
-       xmlns:xacro="http://ros.org/wiki/xacro">
-	<xacro:macro name="frida_adapter" params="parent name *origin">
-		<!-- joint between base_link and torso_link -->
-		<joint name="${name}_adapter_joint" type="fixed" >
-			<insert_block name="origin" />
-			<parent link="${parent}" />
-			<child link="${name}_adapter_link" />
-		</joint>
-		<link name="${name}_adapter_link"/>
-	</xacro:macro>
+<robot xmlns:xacro="http://www.ros.org/wiki/xacro">
+  <xacro:macro name="frida_adapter" params="parent name *origin">
+    <!-- joint between base_link and torso_link -->
+    <joint name="${name}_adapter_joint" type="fixed" >
+      <insert_block name="origin" />
+      <parent link="${parent}" />
+      <child link="${name}_adapter_link" />
+    </joint>
+    <link name="${name}_adapter_link"/>
+  </xacro:macro>
 </robot>

File: frida_description/urdf/frida.urdf.xacro (robot description, xacro)
@@ -1,21 +1,18 @@
 <?xml version="1.0"?>
-<robot xmlns:sensor="http://playerstage.sourceforge.net/gazebo/xmlschema/#sensor"
-       xmlns:controller="http://playerstage.sourceforge.net/gazebo/xmlschema/#controller"
-       xmlns:interface="http://playerstage.sourceforge.net/gazebo/xmlschema/#interface"
-       xmlns:xacro="http://ros.org/wiki/xacro">
-    <!-- this is an empty fake frida for the open source repositories -->
-	<xacro:macro name="frida" params="parent name *origin">
-	<joint name="${name}_left_joint" type="fixed" >
-		<insert_block name="origin" />
-		<parent link="${parent}" />
-		<child link="${name}_left_6_link" />
-	</joint>
-	<link name="${name}_left_6_link"/>
-	<joint name="${name}_right_joint" type="fixed" >
-		<insert_block name="origin" />
-		<parent link="${parent}" />
-		<child link="${name}_right_6_link" />
-	</joint>
-	<link name="${name}_right_6_link"/>
-	</xacro:macro>
+<robot xmlns:xacro="http://www.ros.org/wiki/xacro">
+  <!-- this is an empty fake frida for the open source repositories -->
+  <xacro:macro name="frida" params="parent name *origin">
+  <joint name="${name}_left_joint" type="fixed" >
+    <insert_block name="origin" />
+    <parent link="${parent}" />
+    <child link="${name}_left_6_link" />
+  </joint>
+  <link name="${name}_left_6_link"/>
+  <joint name="${name}_right_joint" type="fixed" >
+    <insert_block name="origin" />
+    <parent link="${parent}" />
+    <child link="${name}_right_6_link" />
+  </joint>
+  <link name="${name}_right_6_link"/>
+  </xacro:macro>
 </robot>

File: prace_gripper_description/urdf/prace_gripper.urdf.xacro (robot description, xacro)
@@ -1,8 +1,5 @@
 <?xml version="1.0"?>
-<robot xmlns:sensor="http://playerstage.sourceforge.net/gazebo/xmlschema/#sensor"
-       xmlns:controller="http://playerstage.sourceforge.net/gazebo/xmlschema/#controller"
-       xmlns:interface="http://playerstage.sourceforge.net/gazebo/xmlschema/#interface"
-       xmlns:xacro="http://ros.org/wiki/xacro">
-	<xacro:macro name="prace_gripper" params="parent name *origin">
-	</xacro:macro>
+<robot xmlns:xacro="http://www.ros.org/wiki/xacro">
+  <xacro:macro name="prace_gripper" params="parent name *origin">
+  </xacro:macro>
 </robot>
