Commit message: update xacro file format

File: frida_description/urdf/camera_holder.urdf.xacro (robot description, xacro)
@@ -1,23 +1,20 @@
 <?xml version="1.0"?>
-<robot xmlns:sensor="http://playerstage.sourceforge.net/gazebo/xmlschema/#sensor"
-       xmlns:controller="http://playerstage.sourceforge.net/gazebo/xmlschema/#controller"
-       xmlns:interface="http://playerstage.sourceforge.net/gazebo/xmlschema/#interface"
-       xmlns:xacro="http://ros.org/wiki/xacro">
-    <!-- this is an empty fake camera_holder for the open source repositories -->
-	<xacro:macro name="teachin_handle" params="parent name *origin">
+<robot xmlns:xacro="http://www.ros.org/wiki/xacro">
+  <!-- this is an empty fake camera_holder for the open source repositories -->
+  <xacro:macro name="teachin_handle" params="parent name *origin">
 <!--
-	<joint name="${name}_left_joint" type="fixed" >
-		<insert_block name="origin" />
-		<parent link="${parent}" />
-		<child link="${name}_left_6_link" />
-	</joint>
-	<link name="${name}_left_6_link"/>
-	<joint name="${name}_right_joint" type="fixed" >
-		<insert_block name="origin" />
-		<parent link="${parent}" />
-		<child link="${name}_right_6_link" />
-	</joint>
-	<link name="${name}_right_6_link"/>
+  <joint name="${name}_left_joint" type="fixed" >
+    <insert_block name="origin" />
+    <parent link="${parent}" />
+    <child link="${name}_left_6_link" />
+  </joint>
+  <link name="${name}_left_6_link"/>
+  <joint name="${name}_right_joint" type="fixed" >
+    <insert_block name="origin" />
+    <parent link="${parent}" />
+    <child link="${name}_right_6_link" />
+  </joint>
+  <link name="${name}_right_6_link"/>
 -->
-	</xacro:macro>
+  </xacro:macro>
 </robot>

File: ur_description/urdf/ur10.urdf.xacro (robot description, xacro)
@@ -1,7 +1,4 @@
-<?xml version="1.0"?>
-<robot xmlns:sensor="http://playerstage.sourceforge.net/gazebo/xmlschema/#sensor"
-       xmlns:controller="http://playerstage.sourceforge.net/gazebo/xmlschema/#controller"
-       xmlns:interface="http://playerstage.sourceforge.net/gazebo/xmlschema/#interface"
-       xmlns:xacro="http://ros.org/wiki/xacro">
+<?xml version="1.0" ?>
+<robot xmlns:xacro="http://www.ros.org/wiki/xacro">
   <xacro:macro name="ur10_robot" params="prefix">
   <link name="${prefix}base_link" />

File: ur_description/urdf/ur10_robot.urdf.xacro (robot description, xacro)
@@ -1,10 +1,7 @@
-<?xml version="1.0"?>
-<robot xmlns:sensor="http://playerstage.sourceforge.net/gazebo/xmlschema/#sensor"
-       xmlns:controller="http://playerstage.sourceforge.net/gazebo/xmlschema/#controller"
-       xmlns:interface="http://playerstage.sourceforge.net/gazebo/xmlschema/#interface"
-       xmlns:xacro="http://playerstage.sourceforge.net/gazebo/xmlschema/#interface"
+<?xml version="1.0" ?>
+<robot xmlns:xacro="http://www.ros.org/wiki/xacro"
        name="ur10" >
   <!-- ur10 -->
-  <include filename="$(find ur_description)/urdf/ur10.urdf.xacro" />
+  <xacro:include filename="$(find ur_description)/urdf/ur10.urdf.xacro" />
   <!-- arm -->
   <xacro:ur10_robot prefix="">

File: ur_description/urdf/ur5.urdf.xacro (robot description, xacro)
@@ -1,7 +1,4 @@
-<?xml version="1.0"?>
-<robot xmlns:sensor="http://playerstage.sourceforge.net/gazebo/xmlschema/#sensor"
-       xmlns:controller="http://playerstage.sourceforge.net/gazebo/xmlschema/#controller"
-       xmlns:interface="http://playerstage.sourceforge.net/gazebo/xmlschema/#interface"
-       xmlns:xacro="http://ros.org/wiki/xacro">
+<?xml version="1.0" ?>
+<robot xmlns:xacro="http://www.ros.org/wiki/xacro">
   <xacro:macro name="ur5_robot" params="prefix">
   <link name="${prefix}base_link" />

File: ur_description/urdf/ur5_robot.urdf.xacro (robot description, xacro)
@@ -1,10 +1,7 @@
-<?xml version="1.0"?>
-<robot xmlns:sensor="http://playerstage.sourceforge.net/gazebo/xmlschema/#sensor"
-       xmlns:controller="http://playerstage.sourceforge.net/gazebo/xmlschema/#controller"
-       xmlns:interface="http://playerstage.sourceforge.net/gazebo/xmlschema/#interface"
-       xmlns:xacro="http://playerstage.sourceforge.net/gazebo/xmlschema/#interface"
+<?xml version="1.0" ?>
+<robot xmlns:xacro="http://www.ros.org/wiki/xacro"
        name="ur5" >
   <!-- ur5 -->
-  <include filename="$(find ur_description)/urdf/ur5.urdf.xacro" />
+  <xacro:include filename="$(find ur_description)/urdf/ur5.urdf.xacro" />
   <!-- arm -->
   <xacro:ur5_robot prefix="">
